Commit message: Update mir_description

File: mir_description/urdf/mir100_macro.xacro (robot description, xacro)
@@ -1,11 +1,12 @@
 <?xml version="1.0"?>
 <robot xmlns:xacro="http://ros.org/wiki/xacro">
-  <xacro:include filename="$(find mir_description)/urdf/include/common_properties.urdf.xacro" />
-  <xacro:include filename="$(find mir_description)/urdf/include/imu.gazebo.urdf.xacro" />
-  <xacro:include filename="$(find mir_description)/urdf/include/mir_100.gazebo.xacro" />
-  <xacro:include filename="$(find mir_description)/urdf/include/mir_100.transmission.xacro" />
-  <xacro:include filename="$(find mir_description)/urdf/include/sick_s300.urdf.xacro" />
-  <xacro:include filename="$(find mir_description)/urdf/include/wheel.urdf.xacro" />
-  <xacro:include filename="$(find mir_description)/urdf/include/caster.urdf.xacro" />
+  <!-- MACROS -->
+  <xacro:include filename="$(find mir_description)/urdf/properties/inertial_macro.xacro" />
+  <xacro:include filename="$(find mir_description)/urdf/properties/material_macro.xacro" />
+  <xacro:include filename="$(find mir_description)/urdf/structures/caster_wheel_macro.xacro" />
+  <xacro:include filename="$(find mir_description)/urdf/structures/drive_wheel_macro.xacro" />
+  <xacro:include filename="$(find mir_description)/urdf/sensors/imu_macro.xacro" />
+  <xacro:include filename="$(find mir_description)/urdf/sensors/sick_s300_macro.xacro" />
+  <!-- PROPERTIES -->
   <xacro:property name="deg_to_rad" value="0.017453293" />
   <!-- The inertia for the MiR platform is intentionally chosen to be smaller than
@@ -39,5 +40,6 @@
   <xacro:property name="mir_100_base_mass" value="66.96" />
   <xacro:property name="imu_stdev" value="0.00017" />
-  <xacro:macro name="mir_100" params="prefix ns">
+  <!-- MiR100 -->
+  <xacro:macro name="mir100" params="prefix ns">
     <link name="${prefix}base_footprint" />
     <joint name="${prefix}base_joint" type="fixed">
@@ -53,5 +55,5 @@
         <origin xyz="${mir_100_act_wheel_dx} 0 0" rpy="0 0 0" />
         <geometry>
-          <mesh filename="package://mir_description/meshes/visual/mir_100_base.stl" />
+          <mesh filename="package://mir_description/meshes/structures/mir100_chassis/mir100_chassis_visual.stl" />
         </geometry>
         <xacro:insert_block name="material_white" />
@@ -60,5 +62,5 @@
         <origin xyz="${mir_100_act_wheel_dx} 0 0" rpy="0 0 0" />
         <geometry>
-          <mesh filename="package://mir_description/meshes/collision/mir_100_base.stl" />
+          <mesh filename="package://mir_description/meshes/structures/mir100_chassis/mir100_chassis_collision.stl" />
         </geometry>
       </collision>
@@ -119,6 +121,6 @@
     <link name="${prefix}us_2_frame" />
     <!-- wheels -->
-    <xacro:actuated_wheel prefix="${prefix}" locationprefix="left" locationright="-1"/>
-    <xacro:actuated_wheel prefix="${prefix}" locationprefix="right" locationright="1"/>
+    <xacro:drive_wheel prefix="${prefix}" locationprefix="left" locationright="-1"/>
+    <xacro:drive_wheel prefix="${prefix}" locationprefix="right" locationright="1"/>
     <xacro:caster_wheel prefix="${prefix}" ns="${ns}" locationprefix="fl" locationright="-1" wheel_base_dx="${mir_100_front_caster_wheel_base_dx}"/>
     <xacro:caster_wheel prefix="${prefix}" ns="${ns}" locationprefix="fr" locationright="1" wheel_base_dx="${mir_100_front_caster_wheel_base_dx}"/>
@@ -140,5 +142,4 @@
     </joint>
     <link name="${prefix}surface_mount"/>
-    <xacro:mir_100_wheel_transmissions prefix="${prefix}"/>
   </xacro:macro>
 </robot>

File: mir_description/urdf/sensors/imu_macro.xacro (robot description, xacro)
@@ -17,5 +17,5 @@
         <update_rate>${update_rate}</update_rate>
         <visualize>true</visualize>
-        <frame_id>${imu_frame}</frame_id>
+        <gz_frame_id>${imu_frame}</gz_frame_id>
         <topic>${imu_topic}</topic>
         <imu>

File: mir_description/urdf/sensors/sick_s300_macro.xacro (robot description, xacro)
@@ -1,5 +1,6 @@
 <?xml version="1.0"?>
 <robot xmlns:xacro="http://ros.org/wiki/xacro">
-  <xacro:include filename="$(find mir_description)/urdf/include/common_properties.urdf.xacro" />
+  <xacro:include filename="$(find mir_description)/urdf/properties/inertial_macro.xacro" />
+  <xacro:include filename="$(find mir_description)/urdf/properties/material_macro.xacro" />
   <xacro:property name="laser_x" value="0.156" />
   <xacro:property name="laser_y" value="0.155" />
@@ -11,5 +12,5 @@
         <origin xyz="0.0 0.0 0.0" rpy="${pi} 0 0" />
         <geometry>
-          <mesh filename="package://mir_description/meshes/visual/sick_lms-100.stl" />
+          <mesh filename="package://mir_description/meshes/sensors/sick_lms_100/sick_lms_100_visual.stl" />
         </geometry>
         <!-- <xacro:insert_block name="material_yellow" /> -->
@@ -19,5 +20,5 @@
         <origin xyz="0.0 0.0 0.0" rpy="${pi} 0 0" />
         <geometry>
-          <mesh filename="package://mir_description/meshes/visual/sick_lms-100.stl" />
+          <mesh filename="package://mir_description/meshes/sensors/sick_lms_100/sick_lms_100_visual.stl" />
         </geometry>
       </collision>
@@ -29,10 +30,8 @@
       <!-- <material value="Gazebo/Yellow" /> -->
       <material value="Gazebo/FlatBlack" />
-      <sensor type="gpu_lidar" name="${prefix}${link}">
+      <sensor type="ray" name="${prefix}${link}">
         <visualize>false</visualize>
         <update_rate>12.5</update_rate>
-        <gz_frame_id>${prefix}${link}</gz_frame_id>
-        <topic>${prefix}${topic}</topic>
-        <lidar>
+        <ray>
           <scan>
             <horizontal>
@@ -45,5 +44,5 @@
           <range>
             <min>0.05</min>
-            <max>8.0</max>
+            <max>29.0</max>
             <resolution>0.01</resolution>
           </range>
@@ -56,12 +55,7 @@
             <stddev>0.01</stddev>
           </noise>
-        </lidar>
-        <!-- <plugin name="gazebo_ros_${link}_controller" type="libgazebo_ros_ray_sensor.so">
-          <ros>
-            <remapping>~/out:=${prefix}${topic}</remapping>
-          </ros>
-          <output_type>sensor_msgs/LaserScan</output_type>
-          <frame_name>${prefix}${link}</frame_name>
-        </plugin> -->
+        </ray>
+        <topic>${prefix}${topic}</topic>
+        <gz_frame_id>${prefix}${link}</gz_frame_id>
       </sensor>
     </gazebo>

File: mir_description/urdf/structures/caster_wheel_macro.xacro (robot description, xacro)
@@ -1,21 +1,17 @@
 <?xml version="1.0"?>
 <robot xmlns:xacro="http://ros.org/wiki/xacro">
-  <xacro:include filename="$(find mir_description)/urdf/include/common_properties.urdf.xacro" />
+  <xacro:include filename="$(find mir_description)/urdf/properties/inertial_macro.xacro" />
+  <xacro:include filename="$(find mir_description)/urdf/properties/material_macro.xacro" />
   <xacro:macro name="caster_wheel" params="prefix ns locationprefix locationright wheel_base_dx">
     <!-- caster hub -->
     <joint name="${prefix}${locationprefix}_caster_rotation_joint" type="continuous">
-      <origin xyz="${wheel_base_dx} ${-mir_100_caster_wheel_base_dy * locationright} ${mir_100_caster_wheel_base_dz}" rpy="0 0 0" />
+      <origin
+        xyz="${wheel_base_dx} ${-mir_100_caster_wheel_base_dy * locationright} ${mir_100_caster_wheel_base_dz}"
+        rpy="0 0 0" />
       <parent link="${prefix}base_link" />
       <child link="${prefix}${locationprefix}_caster_rotation_link" />
       <axis xyz="0 0 1" />
-      <dynamics damping="0.0" friction="0.5"/>
+      <dynamics damping="0.0" friction="0.5" />
     </joint>
-    <gazebo>
-      <plugin filename="gz-sim-joint-state-publisher-system" name="gz::sim::systems::JointStatePublisher">
-        <namespace>${ns}</namespace>
-        <topic>joint_states</topic>
-        <joint_name>${prefix}${locationprefix}_caster_rotation_joint</joint_name>
-      </plugin>
-    </gazebo>
     <link name="${prefix}${locationprefix}_caster_rotation_link">
       <inertial>
@@ -34,5 +30,5 @@
         <origin xyz="0 0 0" rpy="0 0 0" />
         <geometry>
-          <mesh filename="package://mir_description/meshes/visual/caster_wheel_base.stl" />
+          <mesh filename="package://mir_description/meshes/structures/caster_housing/caster_housing_visual.stl" />
         </geometry>
         <xacro:insert_block name="material_silver" />
@@ -41,27 +37,20 @@
         <origin xyz="0 0 0" rpy="0 0 0" />
         <geometry>
-          <mesh filename="package://mir_description/meshes/collision/caster_wheel_base.stl" />
+          <mesh filename="package://mir_description/meshes/structures/caster_housing/caster_housing_collision.stl" />
         </geometry>
       </collision>
     </link>
-    <gazebo reference="${prefix}${locationprefix}_caster_rotation_link">
-      <material>Gazebo/Grey</material>
-    </gazebo>
     <!-- caster wheel -->
     <joint name="${prefix}${locationprefix}_caster_wheel_joint" type="continuous">
-      <origin xyz="${mir_100_caster_wheel_dx} ${-mir_100_caster_wheel_dy * locationright} ${mir_100_caster_wheel_dz}" rpy="0 0 0" />
+      <origin
+        xyz="${mir_100_caster_wheel_dx} ${-mir_100_caster_wheel_dy * locationright} ${mir_100_caster_wheel_dz}"
+        rpy="0 0 0" />
       <parent link="${prefix}${locationprefix}_caster_rotation_link" />
       <child link="${prefix}${locationprefix}_caster_wheel_link" />
       <axis xyz="0 1 0" />
     </joint>
-    <gazebo>
-      <plugin filename="gz-sim-joint-state-publisher-system" name="gz::sim::systems::JointStatePublisher">
-        <namespace>${ns}</namespace>
-        <topic>joint_states</topic>
-        <joint_name>${prefix}${locationprefix}_caster_wheel_joint</joint_name>
-      </plugin>
-    </gazebo>
     <link name="${prefix}${locationprefix}_caster_wheel_link">
-      <xacro:cylinder_inertial mass="${mir_100_caster_wheel_mass}" radius="${mir_100_caster_wheel_radius}" length="${mir_100_caster_wheel_width}">
+      <xacro:cylinder_inertial mass="${mir_100_caster_wheel_mass}"
+        radius="${mir_100_caster_wheel_radius}" length="${mir_100_caster_wheel_width}">
         <origin xyz="0 0 0" rpy="${0.5 * pi} 0 0" />
       </xacro:cylinder_inertial>
@@ -69,5 +58,5 @@
         <origin xyz="0 0 0" rpy="0 0 0" />
         <geometry>
-          <mesh filename="package://mir_description/meshes/visual/wheel.stl" />
+          <mesh filename="package://mir_description/meshes/structures/wheel/wheel.stl" />
         </geometry>
         <xacro:insert_block name="material_dark_grey" />
@@ -80,36 +69,33 @@
       </collision>
     </link>
-    <gazebo reference="${prefix}${locationprefix}_caster_wheel_link">
-      <material>Gazebo/DarkGrey</material>
-    </gazebo>
     <!-- set the gazebo friction parameters for the wheels -->
     <gazebo reference="${prefix}${locationprefix}_caster_wheel_link">
       <collision name="${prefix}${locationprefix}_caster_wheel_link_collision">
         <surface>
-            <friction>
-              <ode>
-                <mu>1.0</mu>
-                <mu2>1.0</mu2>
-                <fdir1>0 0 1</fdir1>
-                <slip1>0.0</slip1>
-                <slip2>0.5</slip2>
-              </ode>
-              <!-- <torsional>
+          <friction>
+            <ode>
+              <mu>1.0</mu>
+              <mu2>1.0</mu2>
+              <fdir1>0 0 1</fdir1>
+              <slip1>0.0</slip1>
+              <slip2>0.5</slip2>
+            </ode>
+            <!-- <torsional>
                 <coefficient>1.0</coefficient>
                 <use_patch_radius>false</use_patch_radius>
                 <surface_radius>${mir_100_caster_wheel_radius}</surface_radius>
               </torsional> -->
-            </friction>
-            <contact>
-              <ode>
-                <!-- <soft_cfm>0.0</soft_cfm>
+          </friction>
+          <contact>
+            <ode>
+              <!-- <soft_cfm>0.0</soft_cfm>
                 <soft_erp>0.2</soft_erp> -->
-                <kp>100000000.0</kp>
-                <!--<kd>1.0</kd> -->
-                <!-- <max_vel>1.0</max_vel> -->
-                <min_depth>0.0</min_depth>
-              </ode>
-            </contact>
-          </surface>
+              <kp>100000000.0</kp>
+              <!--<kd>1.0</kd> -->
+              <!-- <max_vel>1.0</max_vel> -->
+              <min_depth>0.0</min_depth>
+            </ode>
+          </contact>
+        </surface>
       </collision>
     </gazebo>

File: mir_description/urdf/structures/drive_wheel_macro.xacro (robot description, xacro)
@@ -1,6 +1,7 @@
 <?xml version="1.0"?>
 <robot xmlns:xacro="http://ros.org/wiki/xacro">
-  <xacro:include filename="$(find mir_description)/urdf/include/common_properties.urdf.xacro" />
-  <xacro:macro name="actuated_wheel" params="prefix  locationprefix locationright">
+  <xacro:include filename="$(find mir_description)/urdf/properties/inertial_macro.xacro" />
+  <xacro:include filename="$(find mir_description)/urdf/properties/material_macro.xacro" />
+  <xacro:macro name="drive_wheel" params="prefix locationprefix locationright">
     <joint name="${prefix}${locationprefix}_wheel_joint" type="continuous">
       <origin xyz="0.0 ${-mir_100_act_wheel_dy * locationright} ${mir_100_act_wheel_radius}" rpy="0 0 0" />
@@ -21,5 +22,5 @@
         <origin xyz="0 0 0" rpy="0 0 0" />
         <geometry>
-          <mesh filename="package://mir_description/meshes/visual/wheel.stl" />
+          <mesh filename="package://mir_description/meshes/structures/wheel/wheel.stl" />
         </geometry>
         <xacro:insert_block name="material_dark_grey" />
@@ -32,7 +33,4 @@
       </collision>
     </link>
-    <gazebo reference="${prefix}${locationprefix}_wheel_link">
-      <material>Gazebo/DarkGrey</material>
-    </gazebo>
     <!-- set the gazebo friction parameters for the wheels -->
     <gazebo reference="${prefix}${locationprefix}_wheel_link">
