Commit message: Change name of wheel joints

File: mir_description/urdf/structures/drive_wheel_macro.xacro (robot description, xacro)
@@ -4,5 +4,5 @@
   <xacro:include filename="$(find mir_description)/urdf/properties/material_macro.xacro" />
   <xacro:macro name="drive_wheel" params="prefix locationprefix locationright">
-    <joint name="${prefix}${locationprefix}_wheel_joint" type="continuous">
+    <joint name="${prefix}${locationprefix}_drive_wheel_joint" type="continuous">
       <origin xyz="0.0 ${-mir_100_act_wheel_dy * locationright} ${mir_100_act_wheel_radius}" rpy="0 0 0" />
       <parent link="${prefix}base_link" />
