Commit message: Update mir_gazebo

File: mir_gazebo/urdf/mocks/diff_drive_mock.xacro (robot description, xacro)
@@ -1,19 +1,24 @@
 <?xml version="1.0"?>
-<robot xmlns:xacro="http://ros.org/wiki/xacro">
-  <xacro:macro name="mir_100_wheel_transmission" params="prefix locationprefix">
-    <transmission name="${prefix}${locationprefix}_wheel_trans">
-      <type>transmission_interface/SimpleTransmission</type>
-      <joint name="${prefix}${locationprefix}_wheel_joint">
-        <hardwareInterface>hardware_interface/VelocityJointInterface</hardwareInterface>
-      </joint>
-      <actuator name="${prefix}${locationprefix}_wheel_motor">
-        <hardwareInterface>hardware_interface/VelocityJointInterface</hardwareInterface>
-        <mechanicalReduction>1</mechanicalReduction>
-      </actuator>
-    </transmission>
-  </xacro:macro>
-  <xacro:macro name="mir_100_wheel_transmissions" params="prefix">
-    <xacro:mir_100_wheel_transmission prefix="${prefix}" locationprefix="left"/>
-    <xacro:mir_100_wheel_transmission prefix="${prefix}" locationprefix="right"/>
-  </xacro:macro>
+<robot xmlns:xacro="http://www.ros.org/wiki/xacro">
+  <ros2_control name="GazeboSystem" type="system">
+    <hardware>
+      <plugin>gz_ros2_control/GazeboSimSystem</plugin>
+    </hardware>
+    <joint name="left_drive_wheel_joint">
+      <command_interface name="velocity">
+        <param name="min">-1</param>
+        <param name="max">1</param>
+      </command_interface>
+      <state_interface name="position" />
+      <state_interface name="velocity" />
+    </joint>
+    <joint name="right_drive_wheel_joint">
+      <command_interface name="velocity">
+        <param name="min">-1</param>
+        <param name="max">1</param>
+      </command_interface>
+      <state_interface name="position" />
+      <state_interface name="velocity" />
+    </joint>
+  </ros2_control>
 </robot>

File: mir_gazebo/urdf/plugins/ros2_control_plugin.xacro (robot description, xacro)
@@ -1,15 +1,23 @@
 <?xml version="1.0"?>
 <robot xmlns:xacro="http://ros.org/wiki/xacro">
-  <xacro:macro name="controller_plugin_gazebo" params="robot_namespace">
-    <gazebo>
-      <plugin filename="gz_ros2_control-system" name="gz_ros2_control::GazeboSimROS2ControlPlugin">
-        <robot_param>robot_description</robot_param>
-        <robot_param_node>robot_state_publisher</robot_param_node>
-        <xacro:unless value="${robot_namespace == ''}">
-          <robot_namespace>${robot_namespace}</robot_namespace>
-        </xacro:unless>
-        <control_period>0.001</control_period>
-      </plugin>
-    </gazebo>
-  </xacro:macro>
+  <gazebo>
+    <plugin
+      filename="gz_ros2_control-system"
+      name="gz_ros2_control::GazeboSimROS2ControlPlugin"
+    >
+      <!-- <xacro:unless value="${robot_namespace == ''}">
+        <robot_namespace>${robot_namespace}</robot_namespace>
+      </xacro:unless>
+      <control_period>0.001</control_period> -->
+      <robot_param>robot_description</robot_param>
+      <robot_param_node>robot_state_publisher</robot_param_node>
+      <parameters>$(find mir_control)/config/mir_controllers.yaml</parameters>
+      <controller_manager_name>controller_manager</controller_manager_name>
+      <ros>
+        <!-- <namespace>mir100</namespace> -->
+        <!-- <remapping>/mir100/robot_description:=/robot_description</remapping> -->
+        <!-- <remapping>/robot_description:=/robot_description_full</remapping> -->
+      </ros>
+    </plugin>
+  </gazebo>
 </robot>
