Commit message: Update mir_description

File: mir_description/urdf/include/imu_macro.xacro (robot description, xacro)
@@ -1,22 +1,30 @@
 <?xml version="1.0"?>
 <robot xmlns:xacro="http://ros.org/wiki/xacro">
-  <!-- If tf_prefix is given, use "frame tf_prefix/imu_frame", else "imu_frame" -->
-  <xacro:arg name="tf_prefix" default="" />
-  <xacro:property name="tf_prefix" value="$(arg tf_prefix)" />
-  <xacro:if value="${tf_prefix == ''}">
-      <xacro:property name="imu_frame" value="imu_frame" />
-  </xacro:if>
-  <xacro:unless value="${tf_prefix == ''}">
-      <xacro:property name="imu_frame" value="$(arg tf_prefix)/imu_frame" />
-  </xacro:unless>
-  <xacro:macro name="imu_gazebo" params="link imu_topic update_rate stdev">
-    <gazebo reference="${link}">
+  <xacro:property name="imu_topic" value="imu_data" />
+  <xacro:property name="imu_update_rate" value="50.0" />
+  <xacro:property name="imu_stdev" value="0.00017" />
+  <xacro:macro name="imu" params="prefix parent *origin">
+    <joint name="${prefix}imu_joint" type="fixed">
+      <parent link="${parent}" />
+      <child link="${prefix}imu_link" />
+      <xacro:insert_block name="origin" />  <!-- same as real MiR -->
+    </joint>
+    <link name="${prefix}imu_link" />
+    <!-- Create an alias for imu_link. This is necessary because the real MiR's
+         TF has imu_link, but the imu_data topic is published in the imu_frame
+         frame. -->
+    <joint name="${prefix}imu_frame_joint" type="fixed">
+      <parent link="${prefix}imu_link" />
+      <child link="${prefix}imu_frame" />
+    </joint>
+    <link name="${prefix}imu_frame" />
+    <gazebo reference="${prefix}imu_link">
       <gravity>true</gravity>
       <sensor name="imu_sensor" type="imu">
         <always_on>true</always_on>
-        <update_rate>${update_rate}</update_rate>
+        <update_rate>${imu_update_rate}</update_rate>
         <visualize>true</visualize>
-        <frame_id>${imu_frame}</frame_id>
-        <topic>${imu_topic}</topic>
+        <gz_frame_id>${prefix}imu_frame</gz_frame_id>
+        <topic>${prefix}${imu_topic}</topic>
         <imu>
           <angular_velocity>
@@ -24,5 +32,5 @@
               <noise type="gaussian">
                 <mean>0.0</mean>
-                <stddev>${stdev}</stddev>
+                <stddev>${imu_stdev}</stddev>
                 <bias_mean>0.0000075</bias_mean>
                 <bias_stddev>0.0000008</bias_stddev>
@@ -32,5 +40,5 @@
               <noise type="gaussian">
                 <mean>0.0</mean>
-                <stddev>${stdev}</stddev>
+                <stddev>${imu_stdev}</stddev>
                 <bias_mean>0.0000075</bias_mean>
                 <bias_stddev>0.0000008</bias_stddev>
@@ -40,5 +48,5 @@
               <noise type="gaussian">
                 <mean>0.0</mean>
-                <stddev>${stdev}</stddev>
+                <stddev>${imu_stdev}</stddev>
                 <bias_mean>0.0000075</bias_mean>
                 <bias_stddev>0.0000008</bias_stddev>
@@ -50,5 +58,5 @@
               <noise type="gaussian">
                 <mean>0.0</mean>
-                <stddev>${stdev}</stddev>
+                <stddev>${imu_stdev}</stddev>
                 <bias_mean>0.1</bias_mean>
                 <bias_stddev>0.001</bias_stddev>
@@ -58,5 +66,5 @@
               <noise type="gaussian">
                 <mean>0.0</mean>
-                <stddev>${stdev}</stddev>
+                <stddev>${imu_stdev}</stddev>
                 <bias_mean>0.1</bias_mean>
                 <bias_stddev>0.001</bias_stddev>
@@ -66,5 +74,5 @@
               <noise type="gaussian">
                 <mean>0.0</mean>
-                <stddev>${stdev}</stddev>
+                <stddev>${imu_stdev}</stddev>
                 <bias_mean>0.1</bias_mean>
                 <bias_stddev>0.001</bias_stddev>

File: mir_description/urdf/include/sick_s300_macro.xacro (robot description, xacro)
@@ -1,11 +1,17 @@
 <?xml version="1.0"?>
 <robot xmlns:xacro="http://ros.org/wiki/xacro">
-  <xacro:include filename="$(find mir_description)/urdf/include/common_properties.urdf.xacro" />
+  <xacro:include filename="$(find mir_description)/urdf/include/inertial_macros.xacro" />
+  <xacro:include filename="$(find mir_description)/urdf/include/material_properties.xacro" />
   <xacro:property name="laser_x" value="0.156" />
   <xacro:property name="laser_y" value="0.155" />
   <xacro:property name="laser_z" value="0.185" />
   <xacro:property name="laser_mass" value="2.0" />
-  <xacro:macro name="sick_s300" params="link topic prefix">
-    <link name="${prefix}${link}">
+  <xacro:macro name="sick_s300" params="prefix parent *origin">
+    <joint name="${prefix}lidar_joint" type="fixed">
+      <parent link="${parent}" />
+      <child link="${prefix}lidar_link" />
+      <xacro:insert_block name="origin" />
+    </joint>
+    <link name="${prefix}lidar_link">
       <visual>
         <origin xyz="0.0 0.0 0.0" rpy="${pi} 0 0" />
@@ -26,13 +32,11 @@
       </xacro:box_inertial>
     </link>
-    <gazebo reference="${prefix}${link}">
+    <gazebo reference="${prefix}lidar_link">
       <!-- <material value="Gazebo/Yellow" /> -->
-      <material value="Gazebo/FlatBlack" />
-      <sensor type="gpu_lidar" name="${prefix}${link}">
+      <!-- <material value="Gazebo/FlatBlack" /> -->
+      <sensor type="gpu_lidar" name="${prefix}lidar">
         <visualize>false</visualize>
         <update_rate>12.5</update_rate>
-        <gz_frame_id>${prefix}${link}</gz_frame_id>
-        <topic>${prefix}${topic}</topic>
-        <lidar>
+        <ray>
           <scan>
             <horizontal>
@@ -45,5 +49,5 @@
           <range>
             <min>0.05</min>
-            <max>8.0</max>
+            <max>29.0</max>
             <resolution>0.01</resolution>
           </range>
@@ -56,12 +60,7 @@
             <stddev>0.01</stddev>
           </noise>
-        </lidar>
-        <!-- <plugin name="gazebo_ros_${link}_controller" type="libgazebo_ros_ray_sensor.so">
-          <ros>
-            <remapping>~/out:=${prefix}${topic}</remapping>
-          </ros>
-          <output_type>sensor_msgs/LaserScan</output_type>
-          <frame_name>${prefix}${link}</frame_name>
-        </plugin> -->
+        </ray>
+        <topic>${prefix}lidar/scan</topic>
+        <gz_frame_id>${prefix}lidar_link</gz_frame_id>
       </sensor>
     </gazebo>
