Commit message: Update mir_gazebo

File: mir_gazebo/urdf/include/diff_drive_mock.xacro (robot description, xacro)
@@ -1,27 +1,24 @@
 <?xml version="1.0"?>
-<robot xmlns:xacro="http://ros.org/wiki/xacro">
-  <!-- See https://github.com/ros-simulation/gazebo_ros_pkgs/wiki/ROS-2-Migration:-Diff-drive for ros2 information -->
-  <xacro:macro name="diff_controller_plugin_gazebo" params="prefix ns left_wheel_joint right_wheel_joint wheel_separation wheel_radius">
-    <gazebo>
-      <!-- Use gazebo_ros_joint_state_publisher instead of publishWheelJointState -->
-      <plugin filename="gz-sim-joint-state-publisher-system" name="gz::sim::systems::JointStatePublisher">
-        <topic>joint_states</topic> <!--from <ros><remapping> -->
-        <joint_name>${right_wheel_joint}</joint_name>
-        <joint_name>${left_wheel_joint}</joint_name>
-      </plugin>
-      <plugin name="gz::sim::systems::DiffDrive" filename="gz-sim-diff-drive-system">
-        <left_joint>${left_wheel_joint}</left_joint>
-        <right_joint>${right_wheel_joint}</right_joint>
-        <wheel_separation>${wheel_separation}</wheel_separation>
-        <wheel_radius>${wheel_radius}</wheel_radius>
-        <max_linear_acceleration>0.175</max_linear_acceleration>  <!-- computed from <max_linear_acceleration> in the original plugin * wheel_radius-->
-        <topic>${prefix}cmd_vel</topic>
-        <odom_topic>${prefix}odom</odom_topic>
-        <frame_id>${prefix}odom</frame_id>
-        <child_frame_id>${prefix}base_footprint</child_frame_id>
-        <odom_publisher_frequency>1000.0</odom_publisher_frequency>
-        <tf_topic>/tf</tf_topic>
-    </plugin>
-    </gazebo>
-  </xacro:macro>
+<robot xmlns:xacro="http://www.ros.org/wiki/xacro">
+  <ros2_control name="DiffDriveGazeboSystem" type="system">
+    <hardware>
+      <plugin>gz_ros2_control/GazeboSimSystem</plugin>
+    </hardware>
+    <joint name="${mir_prefix}left_drive_wheel_joint">
+      <command_interface name="velocity">
+        <param name="min">-1</param>
+        <param name="max">1</param>
+      </command_interface>
+      <state_interface name="position" />
+      <state_interface name="velocity" />
+    </joint>
+    <joint name="${mir_prefix}right_drive_wheel_joint">
+      <command_interface name="velocity">
+        <param name="min">-1</param>
+        <param name="max">1</param>
+      </command_interface>
+      <state_interface name="position" />
+      <state_interface name="velocity" />
+    </joint>
+  </ros2_control>
 </robot>

File: mir_gazebo/urdf/include/ros2_control_plugin.xacro (robot description, xacro)
@@ -1,15 +1,16 @@
 <?xml version="1.0"?>
 <robot xmlns:xacro="http://ros.org/wiki/xacro">
-  <xacro:macro name="controller_plugin_gazebo" params="robot_namespace">
-    <gazebo>
-      <plugin filename="gz_ros2_control-system" name="gz_ros2_control::GazeboSimROS2ControlPlugin">
-        <robot_param>robot_description</robot_param>
-        <robot_param_node>robot_state_publisher</robot_param_node>
-        <xacro:unless value="${robot_namespace == ''}">
-          <robot_namespace>${robot_namespace}</robot_namespace>
-        </xacro:unless>
-        <control_period>0.001</control_period>
-      </plugin>
-    </gazebo>
-  </xacro:macro>
+  <gazebo>
+    <plugin
+      filename="gz_ros2_control-system"
+      name="gz_ros2_control::GazeboSimROS2ControlPlugin"
+    >
+      <parameters>$(find mir_control)/config/mir_controllers.yaml</parameters>
+      <ros>
+        <!-- <namespace>$(arg mir_namespace)</namespace> -->
+        <!-- <remapping>/robot_description:=/leporino/robot_description</remapping> -->
+        <!-- <remapping>/robot_description:=/robot_description_full</remapping> -->
+      </ros>
+    </plugin>
+  </gazebo>
 </robot>
